File: board.kicad_pcb (KiCad board)
At the start: 2 copper layers, 65 x 65 mm, 45 parts, among them IC1 0915BM15A0001, J1 U.FL, U1 MCP73831, U3 BLE113-A, X1 24MHz 8pF 10ppm -20C +70C, X3 MINI-USB-UX60-MB-5ST

Commit message: Fix minor clearance issues
Routing:
- net (no net): track 37.7 -> 0.00 mm
- net VDD: track 141.8 -> 136.5 mm, vias 6 -> 7
- net GND: track 267.7 -> 265.3 mm
- net /P0_0: track 9.86 -> 7.48 mm
- net /P0_1: track 10.5 -> 8.84 mm
- net Net-(CC1110-DEBUG1-Pad4): track 37.1 -> 38.2 mm
- net Net-(BLE113-DEBUG1-Pad6): track 71.3 -> 70.2 mm
- net Net-(BLE113-DEBUG1-Pad8): track 70.6 -> 69.9 mm
Other:
- outline, holes or cut-outs redrawn
